Commit message: better urdf, description parametrization

File: templates/robosim_description/urdf/include/common_macros.xacro (robot description, xacro)
@@ -2,10 +2,10 @@
 <robot xmlns:xacro="http://wiki.ros.org/xacro">
     <!-- Macros for wheels -->
-    <xacro:macro name="wheel" params="prefix reflect wheel_d wheel_r wheel_mass_kg body_pos_y">
+    <xacro:macro name="wheel" params="prefix reflect robot">
         <link name="${prefix}_wheel">
             <visual>
                 <origin xyz="0 0 0" rpy="0 ${pi/2} 0" />
                 <geometry>
-                <cylinder length="${wheel_d}" radius="${wheel_r}"/>
+                <cylinder length="${robot['wheel']['length']}" radius="${robot['wheel']['radius']}"/>
                 </geometry>
             </visual>
@@ -13,8 +13,8 @@
                 <origin xyz="0 0 0" rpy="0 ${pi/2} 0" />
                 <geometry>
-                <cylinder length="${wheel_d}" radius="${wheel_r}"/>
+                <cylinder length="${robot['wheel']['length']}" radius="${robot['wheel']['radius']}"/>
                 </geometry>
             </collision>
-            <xacro:cylinder_inertial_with_origin radius="${wheel_r}" length="${wheel_d}" mass="${wheel_mass_kg}">
+            <xacro:cylinder_inertial_with_origin radius="${robot['wheel']['radius']}" length="${robot['wheel']['length']}" mass="${robot['body']['mass_kg']}">
                 <origin xyz="0 0 0" rpy="0 ${pi/2} 0" />
             </xacro:cylinder_inertial_with_origin>
@@ -24,5 +24,5 @@
             <parent link="base_link"/>
             <child link="${prefix}_wheel"/>
-            <origin xyz="0 ${reflect*body_pos_y} 0" rpy="0 0 ${pi/2}"/>
+            <origin xyz="0 ${reflect*robot['wheel']['offset_y']} 0" rpy="0 0 ${pi/2}"/>
         </joint>
         <transmission name="${prefix}_wheel_transmission">
@@ -37,10 +37,10 @@
         </transmission>
     </xacro:macro>
-    <xacro:macro name="caster_wheel" params="prefix reflect caster_r caster_pos_x caster_pos_y caster_pos_z">
+    <xacro:macro name="caster_wheel" params="prefix reflect robot">
         <link name="${prefix}_caster_wheel">
             <visual>
                 <origin xyz="0 0 0" rpy="0 0 0" />
                 <geometry>
-                <sphere radius="${caster_r}"/>
+                <sphere radius="${robot['caster']['radius']}"/>
                 </geometry>
             </visual>
@@ -48,5 +48,5 @@
                 <origin xyz="0 0 0" rpy="0 0 0" />
                 <geometry>
-                <sphere radius="${caster_r}"/>
+                <sphere radius="${robot['caster']['radius']}"/>
                 </geometry>
             </collision>
@@ -55,5 +55,5 @@
             <parent link="base_link"/>
             <child link="${prefix}_caster_wheel"/>
-            <origin xyz="${caster_pos_x} ${reflect*caster_pos_y} ${caster_pos_z}" rpy="0 0 0"/>
+            <origin xyz="${robot['caster']['pos_x']} ${reflect*robot['caster']['pos_y']} ${robot['caster']['pos_z']}" rpy="0 0 0"/>
         </joint>
     </xacro:macro>

File: templates/robosim_description/urdf/robosim.urdf.xacro (robot description, xacro)
@@ -1,38 +1,26 @@
 <?xml version="1.0"?>
 <robot xmlns:xacro="http://wiki.ros.org/xacro" name="robosim">
-  <xacro:property name="bodyx" value="@config.body_size_x" />
-  <xacro:property name="bodyy" value="@config.body_size_y" />
-  <xacro:property name="bodyz" value="@config.body_size_z" />
-  <xacro:property name="body_pos_x" value="@config.body_pos_x" />
-  <xacro:property name="body_pos_y" value="${bodyy/2+wheel_d/2+0.01}" />
-  <xacro:property name="body_pos_z" value="@config.body_pos_z" />
-  <xacro:property name="body_mass_kg" value="10.0" />
-  <xacro:property name="wheel_r" value="@config.wheel_size_r" />
-  <xacro:property name="wheel_d" value="@config.wheel_size_d" />
-  <xacro:property name="wheel_mass_kg" value="0.3" />
-  <xacro:property name="caster_r" value="@config.caster_size_r" />
-  <xacro:property name="caster_pos_x" value="@config.caster_pos_x" />
-  <xacro:property name="caster_pos_y" value="@config.caster_pos_y" />
-  <xacro:property name="caster_pos_z" value="@config.caster_pos_z" />
-  <xacro:property name="caster_mass_kg" value="0.1" />
+  <!-- TODO replace naming of robot from param -->
   <xacro:include filename="$(find robosim_description)/urdf/include/common_macros.xacro" />
   <xacro:include filename="$(find robosim_description)/urdf/include/robosim.gazebo.xacro" />
   <xacro:include filename="$(find robosim_description)/urdf/include/inertial.xacro" />
+  <xacro:property name="robot_yaml" value="$(find robosim_description)/config/robot.yaml" />
+  <xacro:property name="robot" value="${xacro.load_yaml(robot_yaml)}"/>
   <!-- Robot base_link -->
   <link name="base_link">
     <visual>
-      <origin xyz="${body_pos_x} 0 ${body_pos_z}" rpy="0 0 0" />
+      <origin xyz="${robot['body']['pos_x']} 0 ${robot['body']['pos_z']}" rpy="0 0 0" />
       <geometry>
-        <box size="${bodyx} ${bodyy} ${bodyz}"/>
+        <box size="${robot['body']['x']} ${robot['body']['y']} ${robot['body']['z']}"/>
       </geometry>
     </visual>
   <collision>
-	  <origin xyz="${body_pos_x} 0 ${body_pos_z}" rpy="0 0 0" />
+	  <origin xyz="${robot['body']['pos_x']} 0 ${robot['body']['pos_z']}" rpy="0 0 0" />
       <geometry>
-        <box size="${bodyx} ${bodyy} ${bodyz}"/>
+        <box size="${robot['body']['x']} ${robot['body']['y']} ${robot['body']['z']}"/>
       </geometry>
   </collision>
-  <xacro:box_inertial_with_origin  x="${bodyx}" y="${bodyy}" z="${bodyz}" mass="${body_mass_kg}">
-    <origin xyz="${body_pos_x} 0 0" rpy="0 0 0" />
+  <xacro:box_inertial_with_origin  x="${robot['body']['x']}" y="${robot['body']['y']}" z="${robot['body']['z']}" mass="${robot['body']['mass_kg']}">
+    <origin xyz="${robot['body']['pos_x']} 0 0" rpy="0 0 0" />
   </xacro:box_inertial_with_origin>
   </link>
@@ -42,11 +30,11 @@
     <parent link="base_footprint"/>
     <child link="base_link"/>
-    <origin xyz="0 0 ${wheel_r}" rpy="0 0 0"/>
+    <origin xyz="0 0 ${robot['wheel']['radius']}" rpy="0 0 0"/>
   </joint>
   <!-- Front wheels -->
-  <xacro:wheel prefix="left" reflect="1" wheel_d="${wheel_d}" wheel_r="${wheel_r}" wheel_mass_kg="${wheel_mass_kg}" body_pos_y="${body_pos_y}"/>
-  <xacro:wheel prefix="right" reflect="-1" wheel_d="${wheel_d}" wheel_r="${wheel_r}" wheel_mass_kg="${wheel_mass_kg}" body_pos_y="${body_pos_y}"/>
+  <xacro:wheel prefix="left" reflect="1" robot="${robot}"/>
+  <xacro:wheel prefix="right" reflect="-1" robot="${robot}"/>
   <!-- Casters -->
-  <xacro:caster_wheel prefix="left" reflect="1" caster_r="${caster_r}" caster_pos_x="${caster_pos_x}" caster_pos_y="${caster_pos_y}" caster_pos_z="${caster_pos_z}"/>
-  <xacro:caster_wheel prefix="right" reflect="-1" caster_r="${caster_r}" caster_pos_x="${caster_pos_x}" caster_pos_y="${caster_pos_y}" caster_pos_z="${caster_pos_z}"/>
+  <xacro:caster_wheel prefix="left" reflect="1" robot="${robot}"/>
+  <xacro:caster_wheel prefix="right" reflect="-1" robot="${robot}"/>
 </robot>
