Commit message: Added lidar

File: templates/robosim_description/urdf/include/sensors_macros.xacro (robot description, xacro)
@@ -1,5 +1,6 @@
 <?xml version="1.0"?>
 <robot xmlns:xacro="http://www.ros.org/wiki/xacro">
-    <xacro:macro name="camera" params=" *joint_origin camera">
+    <!-- Camera -->
+    <xacro:macro name="camera" params=" *joint_origin camera robot">
         <joint name="${camera['name']}_joint" type="fixed">
             <axis xyz="0 1 0" />
@@ -8,5 +9,4 @@
             <child link="${camera['name']}_link"/>
         </joint>
-        <!-- Camera -->
         <link name="${camera['name']}_link">
             <collision>
@@ -60,5 +60,5 @@
                     <alwaysOn>true</alwaysOn>
                     <updateRate>0.0</updateRate>
-                    <cameraName>${camera['name']}</cameraName>
+                    <cameraName>${robot['name']}/${camera['name']}</cameraName>
                     <imageTopicName>image_raw</imageTopicName>
                     <cameraInfoTopicName>camera_info</cameraInfoTopicName>
@@ -74,3 +74,69 @@
         </gazebo>
     </xacro:macro>
+    <!-- Lidar -->
+    <xacro:macro name="lidar" params=" *joint_origin lidar robot">
+        <joint name="${lidar['name']}_joint" type="fixed">
+            <axis xyz="0 1 0" />
+            <xacro:insert_block name="joint_origin" />
+            <parent link="${lidar['parent_link']}"/>
+            <child link="${lidar['name']}_link"/>
+        </joint>
+        <link name="${lidar['name']}_link">
+            <collision>
+                <origin xyz="0 0 0" rpy="0 0 0"/>
+                <geometry>
+                    <cylinder radius="${lidar['radius']}" length="${lidar['length']}"/>
+                </geometry>
+            </collision>
+            <visual>
+                <origin xyz="0 0 0" rpy="0 0 0"/>
+                <geometry>
+                    <cylinder radius="${lidar['radius']}" length="${lidar['length']}"/>
+                </geometry>
+            </visual>
+            <inertial>
+            <mass value="1e-5" />
+            <origin xyz="0 0 0" rpy="0 0 0"/>
+            <inertia ixx="1e-6" ixy="0" ixz="0" iyy="1e-6" iyz="0" izz="1e-6" />
+            </inertial>
+        </link>
+        <gazebo reference="${lidar['name']}_link">
+            <material>Gazebo/Green</material>
+        </gazebo>
+        <gazebo reference="${lidar['name']}_link">
+            <sensor type="gpu_ray" name="${lidar['name']}_sensor">
+            <pose>0 0 0 0 0 0</pose>
+            <visualize>${lidar['lidar_ray_visualize']}</visualize>
+            <update_rate>${lidar['update_rate']}</update_rate>
+            <ray>
+                <scan>
+                <horizontal>
+                    <samples>${lidar['samples']}</samples>
+                    <resolution>${lidar['horizontal_resolution']}</resolution>
+                    <min_angle>${lidar['min_angle']}</min_angle>
+                    <max_angle>${lidar['max_angle']}</max_angle>
+                </horizontal>
+                </scan>
+                <range>
+                    <min>${lidar['min_range']}</min>
+                    <max>${lidar['max_range']}</max>
+                    <resolution>${lidar['range_resolution']}</resolution>
+                </range>
+                <noise>
+                <type>gaussian</type>
+                <!-- Noise parameters based on published spec for Hokuyo laser
+                    achieving "+-30mm" accuracy at range < 10m.  A mean of 0.0m and
+                    stddev of 0.01m will put 99.7% of samples within 0.03m of the true
+                    reading. -->
+                <mean>0.0</mean>
+                <stddev>0.01</stddev>
+                </noise>
+            </ray>
+            <plugin name="gazebo_ros_${lidar['name']}_controller" filename="libgazebo_ros_gpu_laser.so">
+                <topicName>/${robot['name']}/${lidar['name']}/scan</topicName>
+                <frameName>${lidar['name']}_link</frameName>
+            </plugin>
+            </sensor>
+        </gazebo>
+    </xacro:macro>
 </robot>

File: templates/robosim_description/urdf/robosim.urdf.xacro (robot description, xacro)
@@ -42,8 +42,14 @@
   <xacro:caster_wheel prefix="right" reflect="-1" robot="${robot}"/>
   <xacro:if value="${sensors['camera']['enable'] == True }" >
-    <xacro:camera camera="${sensors['camera']}">
+    <xacro:camera camera="${sensors['camera']}" robot="${robot}">
       <origin xyz="${sensors['camera']['x']} ${sensors['camera']['y']} ${sensors['camera']['z']}"
               rpy="${sensors['camera']['roll']} ${sensors['camera']['pitch']} ${sensors['camera']['yaw']}" />
     </xacro:camera>
   </xacro:if>
+  <xacro:if value="${sensors['lidar']['enable'] == True }" >
+    <xacro:lidar lidar="${sensors['lidar']}" robot="${robot}">
+      <origin xyz="${sensors['lidar']['x']} ${sensors['lidar']['y']} ${sensors['lidar']['z']}"
+              rpy="${sensors['lidar']['roll']} ${sensors['lidar']['pitch']} ${sensors['lidar']['yaw']}" />
+    </xacro:lidar>
+  </xacro:if>
 </robot>
